File: docs/KiCad/DIYer_Cutter/DIYer_Cutter.kicad_sch (KiCad schematic)
At the start: 68 parts, among them M1 Stepper_Motor_bipolar, M2 Motor_Servo, Q1 2N2219, SW1 SW_Push, U1 micro:bit, U2 MCP23008-xP, U3 MCP23008-xP, U4 keypad_3x4_matrix, U5 MCP23008-xP, U6 easy_stepper_driver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

Commit message: Updated schematic
Parts:
- removed R55, R56, R57: R_Small_US, symbol Device:R_Small_US
- added R25, R52, R54: R_Small_US, symbol Device:R_Small_US
Connections:
- net +3V3: now also U3.5 (A0), U5.4 (A1); no longer R34.2, R37.2, U5.6 (~{RESET})
- net GND: now also R34.2, R35.1, R36.1, R37.1, U3.3 (A2), U3.4 (A1), U5.3 (A2), U5.5 (A0), R25.2, R52.1, R54.2; no longer R35.2, R36.2
- net at R1.1, U1.20 (P16), U2.6 (~{RESET}): now also R34.1, U3.6 (~{RESET}), U5.6 (~{RESET}), R25.1
- net at DS1.6 (E), U8.16 (B3): now also R54.1
- net at U3.12 (GP2), U4.3 (C1): now also R52.2
- net at U3.13 (GP3), U4.4 (R4): now also R37.2
- net at U3.15 (GP5), U4.6 (R3): now also R36.2
- net at U3.16 (GP6), U4.7 (R2): now also R35.2

Commit message: Probably working devcontainers config
Parts:
- removed R22, R48, R50, R58: R_Small_US, symbol Device:R_Small_US
Connections:
- net +3V3: no longer R49.1, R51.1
- net GND: now also R21.2, R49.1, R51.1; no longer R21.1
- net at U7.9 (3A): now also U5.10 (GP0)
- net at U6.16 (STEP): now also U7.11 (4Y); no longer U5.10 (GP0)
- net at U6.17 (DIR): now also U7.8 (3Y); no longer U5.11 (GP1)
- net at U7.12 (4A): now also U5.11 (GP1)
- net at U3.11 (GP1), U4.2 (R1): now also R52.2
- net at U3.12 (GP2), U4.3 (C1): no longer R52.2
- net at U5.8 (INT): now also R21.1
Other:
- moved on the sheet: M1, M2, U6, U7
